Commit message: basic changes by Hazik

File: urdf/metal_detector_bot.urdf (robot description, URDF)
Before this commit: robot metal_detector_bot, 7 links, 6 joints
Links:
- link Back_left_wheel_link: mass 0.476988947230469 -> 0.49830589190105; geometry collision mesh filename=package://metal_detector_bot_urdf/meshes/Back_left_wheel_li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; visual mesh filename=package://metal_detector_bot_urdf/meshes/Back_left_wheel_li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
- link Back_right_wheel_link: mass 0.476988947230471 -> 0.498305891901051; geometry collision mesh filename=package://metal_detector_bot_urdf/meshes/Back_right_wheel_l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; visual mesh filename=package://metal_detector_bot_urdf/meshes/Back_right_wheel_l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
- link Front_left_wheel_link: mass 0.161301252450132 -> 0.172260974459748; geometry collision mesh filename=package://metal_detector_bot_urdf/meshes/Front_left_wheel_l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; visual mesh filename=package://metal_detector_bot_urdf/meshes/Front_left_wheel_l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
- link Front_right_wheel_link: mass 0.161301252450132 -> 0.172260974459748; geometry collision mesh filename=package://metal_detector_bot_urdf/meshes/Front_right_wheel_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; visual mesh filename=package://metal_detector_bot_urdf/meshes/Front_right_wheel_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
- link Lidar_link: geometry collision mesh filename=package://metal_detector_bot_urdf/meshes/Lidar_link.STL; visual mesh filename=package://metal_detector_bot_urdf/meshes/Lidar_link.STL
- link Metal_detector_plate_link: geometry collision mesh filename=package://metal_detector_bot_urdf/meshes/Metal_detector_pla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; visual mesh filename=package://metal_detector_bot_urdf/meshes/Metal_detector_pla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
- link base_link: geometry collision mesh filename=package://metal_detector_bot_urdf/meshes/base_link.STL; visual mesh filename=package://metal_detector_bot_urdf/meshes/base_link.STL
Joints:
- joint Back_right_wheel_joint: origin xyz=0.483829724966437 -0.329520905371113 0.146370227614205 rpy=1.5707963267949 -1.39626340159546 3.14159265358979 -> xyz=0.48383 -0.32952 0.14637 rpy=1.5708 -1.3963 3.1416
- joint Metal_detector_plate_joint: origin xyz=0.193179132572984 -0.519320905371113 0.109356496732939 rpy=1.5701472443575 -0.00689619877468165 0.0938460523092666 -> xyz=0.19318 -0.51932 0.10936 rpy=1.5701 -0.0068962 0.093846

Commit message: modified the Solidworks Model

File: urdf/metal_detector_bot.urdf (robot description, URDF)
Before this commit: robot metal_detector_bot_urdf, 7 links, 6 joints
Links:
- link Back_left_wheel_link: geometry collision mesh filename=package://metal_detector_bot/meshes/Back_left_wheel_link.STL; visual mesh filename=package://metal_detector_bot/meshes/Back_left_wheel_link.STL
- link Back_right_wheel_link: geometry collision mesh filename=package://metal_detector_bot/meshes/Back_right_wheel_link.S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; visual mesh filename=package://metal_detector_bot/meshes/Back_right_wheel_link.S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
- link Front_left_wheel_link: geometry collision mesh filename=package://metal_detector_bot/meshes/Front_left_wheel_link.S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; visual mesh filename=package://metal_detector_bot/meshes/Front_left_wheel_link.S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
- link Front_right_wheel_link: geometry collision mesh filename=package://metal_detector_bot/meshes/Front_right_wheel_link.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; visual mesh filename=package://metal_detector_bot/meshes/Front_right_wheel_link.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
- link Lidar_link: geometry collision mesh filename=package://metal_detector_bot/meshes/Lidar_link.STL; visual mesh filename=package://metal_detector_bot/meshes/Lidar_link.STL
- link Metal_detector_plate_link: geometry collision mesh filename=package://metal_detector_bot/meshes/Metal_detector_plate_li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; visual mesh filename=package://metal_detector_bot/meshes/Metal_detector_plate_li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
- link base_link: geometry collision mesh filename=package://metal_detector_bot/meshes/base_link.STL; visual mesh filename=package://metal_detector_bot/meshes/base_link.STL

Commit message: Atlast moving

File: urdf/metal_detector_bot.urdf (robot description, URDF)
Before this commit: robot metal_detector_bot, 7 links, 6 joints
Joints:
- joint Back_left_wheel_joint: type revolute -> continuous
- joint Back_right_wheel_joint: type revolute -> continuous
- joint Front_left_wheel_joint: type revolute -> continuous
- joint Front_right_wheel_joint: type revolute -> continuous

Commit message: All errors have been removed, the robot is moving using /cmd_vel

File: urdf/metal_detector_bot.urdf (robot description, URDF)
Before this commit: robot metal_detector_bot, 7 links, 6 joints
Joints:
- joint Back_right_wheel_joint: origin xyz=0.48383 -0.32952 0.14637 rpy=1.5708 -1.3963 3.1416 -> xyz=0.48383 -0.32952 0.14637 rpy=1.5708 0 0
- joint Front_right_wheel_joint: origin xyz=0.13457 -0.31162 0.11335 rpy=1.5708 -0.87933 3.1416 -> xyz=0.13457 -0.31162 0.11335 rpy=1.5708 0 0

Commit message: adding a camera

File: urdf/metal_detector_bot.urdf (robot description, URDF)
Before this commit: robot metal_detector_bot, 7 links, 6 joints
Links:
- added link camera_link, mass 1e-5; collision box size=0.05 0.05 0.05; visual box size=0.05 0.05 0.05
Joints:
- added joint camera_joint: type fixed, parent base_link, child camera_link, origin xyz=0.28528 -0.51932 0.597 rpy=0 0 0, axis 0 1 0

Commit message: Added LIDAR Sensor an Camera: by MBK

File: urdf/metal_detector_bot.urdf (robot description, URDF)
Before this commit: robot metal_detector_bot, 8 links, 7 joints
Links:
- link camera_link: geometry collision box size=0.01 0.01 0.01; visual box size=0.01 0.01 0.01
Joints:
- joint Lidar_joint: origin xyz=0.28528 -0.51932 0.297 rpy=1.5777 -0.00018804 -1.5436 -> xyz=0.28528 -0.51932 0.297 rpy=0 0 0
- joint camera_joint: origin xyz=0.28528 -0.51932 0.597 rpy=0 0 0 -> xyz=0.28528 -0.61932 0.297 rpy=0 0 0
