Commit message: Alhumdulillah complete ROS Navigation Stack has been implemented, the WMR is moving towards rge desired goal location

File: urdf/metal_detector_bot_v2_old.urdf (robot description, URDF)
Before this commit: robot metal_detector_bot, 7 links, 6 joints
Links:
- link Back_left_wheel_link: mass 0.498305891901051 -> 0.49830589190105
- link Back_right_wheel_link: mass 0.498305891901051 -> 0.49830589190105
- link Lidar_link: mass 0.0713753458662671 -> 0.0553297294575326
- link base_link: mass 5.0537397997941 -> 4.90119967390804
Joints:
- joint Back_left_wheel_joint: origin xyz=-0.1766 0.15065 0.019 rpy=-1.5708 -1.3887 0 -> xyz=0.1766 -0.15065 0.019 rpy=1.5708 1.1251 0
- joint Back_right_wheel_joint: origin xyz=-0.1766 -0.15065 0.019 rpy=1.5708 1.322 3.142 -> xyz=0.1766 0.15065 0.019 rpy=-1.5708 -1.3963 3.1416
- joint Ball_caster_left_joint: origin xyz=0.06543 0.07735 -0.04811 rpy=1.5708 0 0 -> xyz=-0.06543 -0.07735 -0.04811 rpy=1.5708 0 0
- joint Ball_caster_right_joint: origin xyz=0.06543 -0.07735 -0.04811 rpy=1.5708 0 0 -> xyz=-0.06543 0.07735 -0.04811 rpy=1.5708 0 0
- joint Lidar_joint: origin xyz=0.0209 0 0.171 rpy=0 0 0 -> xyz=-0.02 0 0.17 rpy=0 0 3.1415
- joint Metal_detector_plate_joint: origin xyz=0.11465 0.00025000000000001 -0.00924999999999999 rpy=1.5707963267949 0 -3.08892219013656 -> xyz=-0.1143 0 -0.008 rpy=1.5708 0 0.0071867
