Commit message: Minor changes to DD Robot

File: urdf/metal_detector_bot_v2.urdf (robot description, URDF)
Before this commit: robot metal_detector_bot_v2, 7 links, 6 joints
Links:
- link Lidar_link: mass 0.0713753510032307 -> 0.0553297294575326
Joints:
- joint Lidar_joint: origin xyz=0.283226064877054 -0.523791886206672 0.315927719919427 rpy=1.57772045120702 -0.000188044043284599 -1.54364562613363 -> xyz=0.28528 -0.51932 0.297 rpy=0 0 0

Commit message: Minor changes to DD Robot

File: urdf/metal_detector_bot_v2.urdf (robot description, URDF)
Before this commit: robot metal_detector_bot_v2, 7 links, 6 joints
Links:
- removed link Lidar_link
Joints:
- removed joint Lidar_joint

Commit message: Minor changes to DD WMR

File: urdf/metal_detector_bot_v2.urdf (robot description, URDF)
Before this commit: robot metal_detector_bot_v2, 6 links, 5 joints
Links:
- added link Lidar_link, mass 0.0553297294575326; collision mesh filename=package://metal_detector_bot/meshes/Lidar_link.STL; visual mesh filename=package://metal_detector_bot/meshes/Lidar_link.STL
Joints:
- added joint Lidar_joint: type revolute, parent base_link, child Lidar_link, origin xyz=0.28528 -0.51932 0.297 rpy=0 0 0, axis 0 1 0, limit lower=0 upper=0 effort=0 velocity=0

Commit message: Minor changes to DD WMR

File: urdf/metal_detector_bot_v2.urdf (robot description, URDF)
Before this commit: robot metal_detector_bot_v2, 7 links, 6 joints
Joints:
- joint Back_left_wheel_joint: type revolute -> continuous
- joint Back_right_wheel_joint: type revolute -> continuous

Commit message: made slight changes in Navigation launch file

File: urdf/metal_detector_bot_v2.urdf (robot description, URDF)
Before this commit: robot metal_detector_bot_v2, 7 links, 6 joints
Joints:
- joint Ball_caster_right_joint: axis 0.332285756911576 -0.806457664239828 -0.489093254443916 -> 0 0 1; origin xyz=0.0534371795012047 -0.413594277716699 0.0530479286982032 rpy=2.65922459739076 0.176277787413547 0.344276962857752 -> xyz=0.0534371795012047 -0.413594277716699 0.0530479286982032 rpy=1.5707963267949 0 0

Commit message: Modifying the DD Model

File: urdf/metal_detector_bot_v2.urdf (robot description, URDF)
Before this commit: robot metal_detector_bot_v2, 7 links, 6 joints
Links:
- removed link Arm_link
- added link Metal_detector_arm_link, mass 0.180271479688744; collision mesh filename=package://metal_detector_bot/meshes/Metal_detector_arm_link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; visual mesh filename=package://metal_detector_bot/meshes/Metal_detector_arm_link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
- link Lidar_link: mass 0.0553297294575326 -> 0.0713753518670423
- link base_link: mass 5.02550363965795 -> 4.90119967390804
Joints:
- removed joint Arm_joint
- added joint Metal_detector_arm_joint: type continuous, parent base_link, child Metal_detector_arm_link, origin xyz=-0.1143 0 -0.008 rpy=1.5708 0 0.0071867, axis 0 1 0
- joint Back_left_wheel_joint: limit lower=0 upper=0 effort=0 velocity=0 -> (none); origin xyz=0.481774530577528 -0.67444223616167 0.165298349849509 rpy=1.5707963267949 0 0 -> xyz=0.1766 -0.15065 0.019 rpy=1.5708 1.1251 0
- joint Back_right_wheel_joint: limit lower=0 upper=0 effort=0 velocity=0 -> (none); origin xyz=0.481774530577528 -0.33399223616167 0.165298349849508 rpy=1.5707963267949 -1.39626340159546 3.14159265358979 -> xyz=0.1766 0.15065 0.019 rpy=-1.5708 -1.3963 3.1416
- joint Ball_caster_left_joint: origin xyz=0.0534371795019374 -0.601142236161636 0.0530479286981914 rpy=1.5707963267949 0 0 -> xyz=-0.06543 -0.07735 -0.04811 rpy=1.5708 0 0
- joint Ball_caster_right_joint: origin xyz=0.0534371795012047 -0.413594277716699 0.0530479286982032 rpy=1.5707963267949 0 0 -> xyz=-0.06543 0.07735 -0.04811 rpy=1.5708 0 0
- joint Lidar_joint: limit lower=0 upper=0 effort=0 velocity=0 -> (none); origin xyz=0.28528 -0.51932 0.297 rpy=0 0 0 -> xyz=-0.0209 0 0.171 rpy=1.5708 0 -1.5436; type revolute -> continuous

Commit message: Adding joint state publisher gazebo plugin in urdf file

File: urdf/metal_detector_bot_v2.urdf (robot description, URDF)
Before this commit: robot metal_detector_bot_v2, 7 links, 6 joints
Joints:
- removed joint Metal_detector_arm_joint
- added joint Metal_detector_plate_joint: type continuous, parent base_link, child Metal_detector_arm_link, origin xyz=-0.1143 0 -0.008 rpy=1.5708 0 0.0071867, axis 0 1 0

Commit message: LIDAR is placed incorrectly need to cotrrect it

File: urdf/metal_detector_bot_v2.urdf (robot description, URDF)
Before this commit: robot metal_detector_bot_v2, 7 links, 6 joints
Links:
- link Lidar_link: mass 0.0713753518670423 -> 0.0553297294575326
Joints:
- joint Lidar_joint: limit (none) -> lower=0 upper=0 effort=0 velocity=0; origin xyz=-0.0209 0 0.171 rpy=1.5708 0 -1.5436 -> xyz=0.28528 -0.51932 0.297 rpy=0 0 0; type continuous -> revolute

Commit message: Map can be built ALhumdulillah everything working fine

File: urdf/metal_detector_bot_v2.urdf (robot description, URDF)
Before this commit: robot metal_detector_bot_v2, 7 links, 6 joints
Joints:
- joint Lidar_joint: origin xyz=0.28528 -0.51932 0.297 rpy=0 0 0 -> xyz=-0.02 0 0.17 rpy=0 0 0

Commit message: changing the LIDAR link from revolute to fixed

File: urdf/metal_detector_bot_v2.urdf (robot description, URDF)
Before this commit: robot metal_detector_bot_v2, 7 links, 6 joints
Joints:
- joint Lidar_joint: limit lower=0 upper=0 effort=0 velocity=0 -> (none); type revolute -> fixed

Commit message: Modifying the LIDAR rpy properties, now it is aligned in RVIZ and Gazebo

File: urdf/metal_detector_bot_v2.urdf (robot description, URDF)
Before this commit: robot metal_detector_bot_v2, 7 links, 6 joints
Joints:
- joint Lidar_joint: origin xyz=-0.02 0 0.17 rpy=0 0 0 -> xyz=-0.02 0 0.17 rpy=0 0 3.1415

Commit message: Updated Aruino code with tf Broadcaster

File: urdf/metal_detector_bot_v2.urdf (robot description, URDF)
Before this commit: robot metal_detector_bot, 7 links, 6 joints
Links:
- removed link Back_left_wheel_link
- removed link Back_right_wheel_link
- added link left_wheel_link, mass 0.498305891901051; collision mesh filename=package://metal_detector_bot/meshes/Back_left_wheel_link.STL; visual mesh filename=package://metal_detector_bot/meshes/Back_left_wheel_link.STL
- added link right_wheel_link, mass 0.498305891901051; collision mesh filename=package://metal_detector_bot/meshes/Back_right_wheel_link.S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; visual mesh filename=package://metal_detector_bot/meshes/Back_right_wheel_link.S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
Joints:
- removed joint Back_left_wheel_joint
- removed joint Back_right_wheel_joint
- added joint left_wheel_joint: type continuous, parent base_link, child left_wheel_link, origin xyz=-0.1766 0.15065 0.019 rpy=-1.5708 -1.3887 0, axis 0 0 1
- added joint right_wheel_joint: type continuous, parent base_link, child right_wheel_link, origin xyz=-0.1766 -0.15065 0.019 rpy=1.5708 1.322 3.142, axis 0 0 1
